File: hardware/bootstrap_exp/bootstrap_exp.kicad_sch (KiCad schematic)
At the start: 32 parts, among them J1 Conn_Coaxial, J2 Conn_Coaxial, U1 OPA810DBV, U2 OPA810DBV, U3 OPA810DBV, U4 OPA810DBV

Commit message: Specify dielectric for input coupling capacitance
Parts:
- C1: value 80p -> 80p/C0G
- gave numbers to parts that had none: 1
Changed lines of the file:
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@@
   (symbol (lib_id "power:GND") (at 69.85 90.17 0) (unit 1)
     (in_bom yes) (on_board yes) (fields_autoplaced)
-    (property "Reference" "#PWR?" (id 0) (at 69.85 96.52 0)
+    (property "Reference" "#PWR0101" (id 0) (at 69.85 96.52 0)
       (effects (font (size 1.27 1.27)) hide)
     )
@@
     (in_bom yes) (on_board yes) (fields_autoplaced)
     (property "Reference" "C1" (id 0) (at 119.38 50.8 90))
-    (property "Value" "80p" (id 1) (at 119.38 53.34 90))
+    (property "Value" "80p/C0G" (id 1) (at 119.38 53.34 90))
     (property "Footprint" "Capacitor_SMD:C_0603_1608Metric" (id 2) (at 115.57 59.3852 0)
       (effects (font (size 1.27 1.27)) hide)
@@
   (symbol (lib_id "Connector:TestPoint") (at 67.31 87.63 90) (mirror x) (unit 1)
     (in_bom yes) (on_board yes)
-    (property "Reference" "TP?" (id 0) (at 62.23 86.36 90)
+    (property "Reference" "TP8" (id 0) (at 62.23 86.36 90)
       (effects (font (size 1.27 1.27)) (justify left))
     )
@@
     )
     (path "/1f1f5a5e-93ba-4083-b840-ba05eefc4082"
-      (reference "#PWR?") (unit 1) (value "GND") (footprint "")
+      (reference "#PWR0101") (unit 1) (value "GND") (footprint "")
     )
     (path "/a7d158f3-55a4-47ef-8947-cfce6892a922"
-      (reference "C1") (unit 1) (value "80p") (footprint "Capacitor_SMD:C_0603_1608Metric")
+      (reference "C1") (unit 1) (value "80p/C0G") (footprint "Capacitor_SMD:C_0603_1608Metric")
     )
     (path "/39c14ccd-4381-4874-b62d-469a6390c321"
@@
     )
     (path "/ebd243f0-1c55-483e-88ff-76d4cdd404f4"
-      (reference "TP?") (unit 1) (value "GND") (footprint "TestPoint:TestPoint_Keystone_5005-5009_Compact")
+      (reference "TP8") (unit 1) (value "GND") (footprint "TestPoint:TestPoint_Keystone_5005-5009_Compact")
     )
     (path "/de13541f-796c-4950-ab90-fb9467a8b0a3"

Commit message: Update OPA810 footprint to SC-70-5, workaround for shortages
Parts:
- U1, U2, U3, U4: footprint Package_TO_SOT_SMD:SOT-23-5 -> Package_TO_SOT_SMD:SOT-353_SC-70-5
Changed lines of the file:
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@@
       (effects (font (size 1.27 1.27)) (justify left))
     )
-    (property "Footprint" "Package_TO_SOT_SMD:SOT-23-5" (id 2) (at 163.83 105.41 0)
+    (property "Footprint" "Package_TO_SOT_SMD:SOT-353_SC-70-5" (id 2) (at 163.83 105.41 0)
       (effects (font (size 1.27 1.27)) (justify left) hide)
     )
@@
       (effects (font (size 1.27 1.27)) (justify left))
     )
-    (property "Footprint" "Package_TO_SOT_SMD:SOT-23-5" (id 2) (at 90.17 63.5 0)
+    (property "Footprint" "Package_TO_SOT_SMD:SOT-353_SC-70-5" (id 2) (at 90.17 63.5 0)
       (effects (font (size 1.27 1.27)) (justify left) hide)
     )
@@
       (effects (font (size 1.27 1.27)) (justify left))
     )
-    (property "Footprint" "Package_TO_SOT_SMD:SOT-23-5" (id 2) (at 149.86 66.04 0)
+    (property "Footprint" "Package_TO_SOT_SMD:SOT-353_SC-70-5" (id 2) (at 149.86 66.04 0)
       (effects (font (size 1.27 1.27)) (justify left) hide)
     )
@@
       (effects (font (size 1.27 1.27)) (justify left))
     )
-    (property "Footprint" "Package_TO_SOT_SMD:SOT-23-5" (id 2) (at 198.12 68.58 0)
+    (property "Footprint" "Package_TO_SOT_SMD:SOT-353_SC-70-5" (id 2) (at 198.12 68.58 0)
       (effects (font (size 1.27 1.27)) (justify left) hide)
     )
@@
     )
     (path "/de13541f-796c-4950-ab90-fb9467a8b0a3"
-      (reference "U1") (unit 1) (value "OPA810DBV") (footprint "Package_TO_SOT_SMD:SOT-23-5")
+      (reference "U1") (unit 1) (value "OPA810DBV") (footprint "Package_TO_SOT_SMD:SOT-353_SC-70-5")
     )
     (path "/638c9b9e-de88-4b55-9faa-cb8dcfa56597"
-      (reference "U2") (unit 1) (value "OPA810DBV") (footprint "Package_TO_SOT_SMD:SOT-23-5")
+      (reference "U2") (unit 1) (value "OPA810DBV") (footprint "Package_TO_SOT_SMD:SOT-353_SC-70-5")
     )
     (path "/ede33817-1483-4791-9634-7ce6965248ce"
-      (reference "U3") (unit 1) (value "OPA810DBV") (footprint "Package_TO_SOT_SMD:SOT-23-5")
+      (reference "U3") (unit 1) (value "OPA810DBV") (footprint "Package_TO_SOT_SMD:SOT-353_SC-70-5")
     )
     (path "/cc42f723-4a9c-4dfc-b268-ac41daaf52ed"
-      (reference "U4") (unit 1) (value "OPA810DBV") (footprint "Package_TO_SOT_SMD:SOT-23-5")
-    )
-  )
+      (reference "U4") (unit 1) (value "OPA810DBV") (footprint "Package_TO_SOT_SMD:SOT-353_SC-70-5")
+    )
+  )

Commit message: Specify MPN and source for every component
Parts:
- C1: value 80p/C0G -> 100p/NP0/1%; MFR (none) -> YAGEO; MPN (none) -> CC0603FRNPO0BN101; Source (none) -> LCSC
- C10, C11, C3, C4, C5, C7, C8, C9: MFR (none) -> Samsung; MPN (none) -> CL10B104KB8NNNC; Source (none) -> LCSC
- C2, C6: footprint Capacitor_SMD:C_0603_1608Metric -> Capacitor_Tantalum_SMD:CP_EIA-3528-12_Kemet-T; MFR (none) -> KEMET; MPN (none) -> T491B106K025AT; Source (none) -> LCSC
- R1, R7: footprint Resistor_SMD:R_0603_1608Metric -> Resistor_SMD:R_0805_2012Metric; MFR (none) -> Panasonic; MPN (none) -> ERA-6AEB49R9V; Source (none) -> Mouser
- R2: MFR (none) -> YAGEO; MPN (none) -> RC0603FR-071KL
- R3, R4: MFR (none) -> YAGEO; MPN (none) -> RC0603FR-071ML
- R5, R6: MFR (none) -> YAGEO; MPN (none) -> RC0603FR-070RL; Source (none) -> LCSC
- TP1, TP2, TP3, TP4, TP5, TP6, TP7, TP8: MFR (none) -> Keystone; MPN (none) -> 5007; Source (none) -> Mouser
- U1, U2, U3, U4: value OPA810DBV -> OPA810; MFR (none) -> TI; MPN (none) -> OPA810IDCKR; Source (none) -> Mouser
Other:
- note added: "100p/NP0/1%: CC0603FRNPO0BN101 22p/NP0/1%: CC0603FRNPO0BN220"

Commit message: Specify source for resistors
Parts:
- R2, R3, R4: Source (none) -> LCSC
Changed lines of the file:
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@@
+      (effects (font (size 1.27 1.27)) hide)
+    )
+    (property "Source" "LCSC" (id 6) (at 130.81 64.77 0)
       (effects (font (size 1.27 1.27)) hide)
     )
@@
       (effects (font (size 1.27 1.27)) hide)
     )
+    (property "Source" "LCSC" (id 6) (at 179.07 77.47 0)
+      (effects (font (size 1.27 1.27)) hide)
+    )
     (pin "1")
     (pin "2")
@@
       (effects (font (size 1.27 1.27)) hide)
     )
+    (property "Source" "LCSC" (id 6) (at 179.07 90.17 0)
+      (effects (font (size 1.27 1.27)) hide)
+    )
